File: Hardware/KiCad Files/Robot_Arm_Shield.sch (KiCad schematic (older format))
At the start: 28 parts, among them P1 Power Input, P10 Motor 3, P11 Motor 2, P12 Motor 1, P13 Motor 0, P2 Analog In 0, P3 Analog In 1, P4 Analog In 2, P5 Analog In 3, P6 Analog In 4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

Commit message: PCB Layout
Placed parts on board and updated some labels. Also added Freetronics files directly into folder. Edited 7805 symbol to allow for easy footprint placement.
Parts:
- C1, C2: footprint (none) -> Capacitors_ThroughHole:C_Radial_D5_L11_P2
- D1: footprint (none) -> Diodes_SMD:DO-214AB_Handsoldering
- R1: value 68 -> 150
- R2, R3, R4: value R -> 10k
Changed lines of the file:
@@
 F 0 "U1" H 2950 954 50  0000 C CNN
 F 1 "LM 7805" H 2800 1350 50  0000 C CNN
-F 2 "" H 2800 1150 50  0000 C CNN
+F 2 "" H 2800 1150 50  0001 C CNN
 F 3 "" H 2800 1150 50  0000 C CNN
 	1    2800 1150
@@
 F 0 "C1" H 2325 1450 50  0000 L CNN
 F 1 "0.33 uF" H 2325 1250 50  0000 L CNN
-F 2 "" H 2300 1350 50  0000 C CNN
+F 2 "Capacitors_ThroughHole:C_Radial_D5_L11_P2" H 2300 1350 50  0001 C CNN
 F 3 "" H 2300 1350 50  0000 C CNN
 	1    2300 1350
@@
 F 0 "C2" H 3325 1450 50  0000 L CNN
 F 1 "0.1 uF" H 3325 1250 50  0000 L CNN
-F 2 "" H 3300 1350 50  0000 C CNN
+F 2 "Capacitors_ThroughHole:C_Radial_D5_L11_P2" H 3300 1350 50  0001 C CNN
 F 3 "" H 3300 1350 50  0000 C CNN
 	1    3300 1350
@@
 F 0 "P1" H 1250 1300 50  0000 C CNN
 F 1 "Power Input" V 1350 1150 50  0000 C CNN
-F 2 "" H 1250 1150 50  0000 C CNN
+F 2 "" H 1250 1150 50  0001 C CNN
 F 3 "" H 1250 1150 50  0000 C CNN
 	1    1250 1150
@@
 F 0 "P9" H 7250 3850 50  0000 C CNN
 F 1 "Motor 4" V 7350 3650 50  0000 C CNN
-F 2 "" H 7250 3650 50  0000 C CNN
+F 2 "" H 7250 3650 50  0001 C CNN
 F 3 "" H 7250 3650 50  0000 C CNN
 	1    7250 3650
@@
 F 0 "P10" H 7250 4400 50  0000 C CNN
 F 1 "Motor 3" V 7350 4200 50  0000 C CNN
-F 2 "" H 7250 4200 50  0000 C CNN
+F 2 "" H 7250 4200 50  0001 C CNN
 F 3 "" H 7250 4200 50  0000 C CNN
 	1    7250 4200
@@
 F 0 "P11" H 7250 4950 50  0000 C CNN
 F 1 "Motor 2" V 7350 4750 50  0000 C CNN
-F 2 "" H 7250 4750 50  0000 C CNN
+F 2 "" H 7250 4750 50  0001 C CNN
 F 3 "" H 7250 4750 50  0000 C CNN
 	1    7250 4750
@@
 F 0 "P12" H 7250 5500 50  0000 C CNN
 F 1 "Motor 1" V 7350 5300 50  0000 C CNN
-F 2 "" H 7250 5300 50  0000 C CNN
+F 2 "" H 7250 5300 50  0001 C CNN
 F 3 "" H 7250 5300 50  0000 C CNN
 	1    7250 5300
@@
 F 0 "P13" H 7250 6050 50  0000 C CNN
 F 1 "Motor 0" V 7350 5850 50  0000 C CNN
-F 2 "" H 7250 5850 50  0000 C CNN
+F 2 "" H 7250 5850 50  0001 C CNN
 F 3 "" H 7250 5850 50  0000 C CNN
 	1    7250 5850
@@
 F 0 "P8" H 7250 3300 50  0000 C CNN
 F 1 "Motor 5" V 7350 3100 50  0000 C CNN
-F 2 "" H 7250 3100 50  0000 C CNN
+F 2 "" H 7250 3100 50  0001 C CNN
 F 3 "" H 7250 3100 50  0000 C CNN
 	1    7250 3100
@@
 F 0 "P6" H 2850 5500 50  0000 C CNN
 F 1 "Analog In 4" V 2950 5300 50  0000 C CNN
-F 2 "" H 2850 5300 50  0000 C CNN
+F 2 "" H 2850 5300 50  0001 C CNN
 F 3 "" H 2850 5300 50  0000 C CNN
 	1    2850 5300
@@
 F 0 "P5" H 2850 4950 50  0000 C CNN
 F 1 "Analog In 3" V 2950 4750 50  0000 C CNN
-F 2 "" H 2850 4750 50  0000 C CNN
+F 2 "" H 2850 4750 50  0001 C CNN
 F 3 "" H 2850 4750 50  0000 C CNN
 	1    2850 4750
@@
 F 0 "P4" H 2850 4400 50  0000 C CNN
 F 1 "Analog In 2" V 2950 4200 50  0000 C CNN
-F 2 "" H 2850 4200 50  0000 C CNN
+F 2 "" H 2850 4200 50  0001 C CNN
 F 3 "" H 2850 4200 50  0000 C CNN
 	1    2850 4200
@@
 F 0 "P3" H 2850 3850 50  0000 C CNN
 F 1 "Analog In 1" V 2950 3650 50  0000 C CNN
-F 2 "" H 2850 3650 50  0000 C CNN
+F 2 "" H 2850 3650 50  0001 C CNN
 F 3 "" H 2850 3650 50  0000 C CNN
 	1    2850 3650
@@
 F 0 "P2" H 2850 3300 50  0000 C CNN
 F 1 "Analog In 0" V 2950 3100 50  0000 C CNN
-F 2 "" H 2850 3100 50  0000 C CNN
+F 2 "" H 2850 3100 50  0001 C CNN
 F 3 "" H 2850 3100 50  0000 C CNN
 	1    2850 3100
@@
 F 0 "P7" H 2850 6050 50  0000 C CNN
 F 1 "Analog In 5" V 2950 5850 50  0000 C CNN
-F 2 "" H 2850 5850 50  0000 C CNN
+F 2 "" H 2850 5850 50  0001 C CNN
 F 3 "" H 2850 5850 50  0000 C CNN
 	1    2850 5850
@@
 F 0 "D1" H 1850 1200 50  0000 C CNN
 F 1 "D_Schottky" H 1850 1000 50  0000 C CNN
-F 2 "" H 1850 1100 50  0000 C CNN
+F 2 "Diodes_SMD:DO-214AB_Handsoldering" H 1850 1100 50  0001 C CNN
 F 3 "" H 1850 1100 50  0000 C CNN
 	1    1850 1100
@@
 F 0 "LED1" H 4050 2100 50  0000 C CNN
 F 1 "Power LED" H 4050 1900 50  0000 C CNN
-F 2 "" H 4050 2000 60  0000 C CNN
+F 2 "" H 4050 2000 60  0001 C CNN
 F 3 "" H 4050 2000 60  0000 C CNN
 	1    4050 2000
@@
 P 4050 1450
 F 0 "R1" V 4130 1450 50  0000 C CNN
-F 1 "68" V 4050 1450 50  0000 C CNN
-F 2 "" H 4050 1450 60  0000 C CNN
+F 1 "150" V 4050 1450 50  0000 C CNN
+F 2 "" H 4050 1450 60  0001 C CNN
 F 3 "" H 4050 1450 60  0000 C CNN
 	1    4050 1450
@@
 F 0 "SW1" H 6000 1260 50  0000 C CNN
 F 1 "Button 0" H 6150 1070 50  0000 C CNN
-F 2 "" H 6150 1150 60  0000 C CNN
+F 2 "" H 6150 1150 60  0001 C CNN
 F 3 "" H 6150 1150 60  0000 C CNN
 	1    6150 1150
@@
 P 6950 1150
 F 0 "R2" V 7030 1150 50  0000 C CNN
-F 1 "R" V 6950 1150 50  0000 C CNN
-F 2 "" H 6950 1150 60  0000 C CNN
+F 1 "10k" V 6950 1150 50  0000 C CNN
+F 2 "" H 6950 1150 60  0001 C CNN
 F 3 "" H 6950 1150 60  0000 C CNN
 	1    6950 1150
@@
 F 0 "SW2" H 6000 1760 50  0000 C CNN
 F 1 "Button 1" H 6150 1570 50  0000 C CNN
-F 2 "" H 6150 1650 60  0000 C CNN
+F 2 "" H 6150 1650 60  0001 C CNN
 F 3 "" H 6150 1650 60  0000 C CNN
 	1    6150 1650
@@
 P 6950 1650
 F 0 "R3" V 7030 1650 50  0000 C CNN
-F 1 "R" V 6950 1650 50  0000 C CNN
-F 2 "" H 6950 1650 60  0000 C CNN
+F 1 "10k" V 6950 1650 50  0000 C CNN
+F 2 "" H 6950 1650 60  0001 C CNN
 F 3 "" H 6950 1650 60  0000 C CNN
 	1    6950 1650
@@
 F 0 "SW3" H 6000 2260 50  0000 C CNN
 F 1 "Button 2" H 6150 2070 50  0000 C CNN
-F 2 "" H 6150 2150 60  0000 C CNN
+F 2 "" H 6150 2150 60  0001 C CNN
 F 3 "" H 6150 2150 60  0000 C CNN
 	1    6150 2150
@@
 P 6950 2150
 F 0 "R4" V 7030 2150 50  0000 C CNN
-F 1 "R" V 6950 2150 50  0000 C CNN
-F 2 "" H 6950 2150 60  0000 C CNN
+F 1 "10k" V 6950 2150 50  0000 C CNN
+F 2 "" H 6950 2150 60  0001 C CNN
 F 3 "" H 6950 2150 60  0000 C CNN
 	1    6950 2150
@@
 F 0 "R5" V 8680 1150 50  0000 C CNN
 F 1 "150" V 8600 1150 50  0000 C CNN
-F 2 "" H 8600 1150 60  0000 C CNN
+F 2 "" H 8600 1150 60  0001 C CNN
 F 3 "" H 8600 1150 60  0000 C CNN
 	1    8600 1150
@@
 F 0 "LED2" H 9200 1250 50  0000 C CNN
 F 1 "Status LED" H 9200 1050 50  0000 C CNN
-F 2 "" H 9200 1150 60  0000 C CNN
+F 2 "" H 9200 1150 60  0001 C CNN
 F 3 "" H 9200 1150 60  0000 C CNN
 	1    9200 1150

Commit message: Finalized Board. Exported Gerbers
Parts:
- added P14: Power Jumper, Pin_Headers:Pin_Header_Straight_1x02, symbol CONN_01X02
- LED1, LED2: footprint (none) -> FT:LED-1206
- P1: footprint (none) -> FT:SCREWTERMINAL-3.5MM-2
- P10, P11, P12, P13, P8, P9: footprint (none) -> Pin_Headers:Pin_Header_Straight_1x03
- P2, P3, P4, P5, P6, P7: footprint (none) -> Socket_Strips:Socket_Strip_Straight_1x03
- R1, R2, R3, R4, R5: footprint (none) -> Resistors_SMD:R_1206_HandSoldering
- SW1, SW2, SW3: footprint (none) -> Buttons_Switches_SMD:SW_SPST_PTS645
- U1: footprint (none) -> FT:DPAK
Connections:
- net 5V: now also P14.1 (P1); no longer SHIELD1.5V
- new net: P14.2 (P2), SHIELD1.5V
Changed lines of the file:
@@
 F 0 "U1" H 2950 954 50  0000 C CNN
 F 1 "LM 7805" H 2800 1350 50  0000 C CNN
-F 2 "" H 2800 1150 50  0001 C CNN
+F 2 "FT:DPAK" H 2800 1150 50  0001 C CNN
 F 3 "" H 2800 1150 50  0000 C CNN
 	1    2800 1150
@@
 F 0 "P1" H 1250 1300 50  0000 C CNN
 F 1 "Power Input" V 1350 1150 50  0000 C CNN
-F 2 "" H 1250 1150 50  0001 C CNN
+F 2 "FT:SCREWTERMINAL-3.5MM-2" H 1250 1150 50  0001 C CNN
 F 3 "" H 1250 1150 50  0000 C CNN
 	1    1250 1150
@@
 F 0 "P9" H 7250 3850 50  0000 C CNN
 F 1 "Motor 4" V 7350 3650 50  0000 C CNN
-F 2 "" H 7250 3650 50  0001 C CNN
+F 2 "Pin_Headers:Pin_Header_Straight_1x03" H 7250 3650 50  0001 C CNN
 F 3 "" H 7250 3650 50  0000 C CNN
 	1    7250 3650
@@
 F 0 "P10" H 7250 4400 50  0000 C CNN
 F 1 "Motor 3" V 7350 4200 50  0000 C CNN
-F 2 "" H 7250 4200 50  0001 C CNN
+F 2 "Pin_Headers:Pin_Header_Straight_1x03" H 7250 4200 50  0001 C CNN
 F 3 "" H 7250 4200 50  0000 C CNN
 	1    7250 4200
@@
 F 0 "P11" H 7250 4950 50  0000 C CNN
 F 1 "Motor 2" V 7350 4750 50  0000 C CNN
-F 2 "" H 7250 4750 50  0001 C CNN
+F 2 "Pin_Headers:Pin_Header_Straight_1x03" H 7250 4750 50  0001 C CNN
 F 3 "" H 7250 4750 50  0000 C CNN
 	1    7250 4750
@@
 F 0 "P12" H 7250 5500 50  0000 C CNN
 F 1 "Motor 1" V 7350 5300 50  0000 C CNN
-F 2 "" H 7250 5300 50  0001 C CNN
+F 2 "Pin_Headers:Pin_Header_Straight_1x03" H 7250 5300 50  0001 C CNN
 F 3 "" H 7250 5300 50  0000 C CNN
 	1    7250 5300
@@
 F 0 "P13" H 7250 6050 50  0000 C CNN
 F 1 "Motor 0" V 7350 5850 50  0000 C CNN
-F 2 "" H 7250 5850 50  0001 C CNN
+F 2 "Pin_Headers:Pin_Header_Straight_1x03" H 7250 5850 50  0001 C CNN
 F 3 "" H 7250 5850 50  0000 C CNN
 	1    7250 5850
@@
 F 0 "P8" H 7250 3300 50  0000 C CNN
 F 1 "Motor 5" V 7350 3100 50  0000 C CNN
-F 2 "" H 7250 3100 50  0001 C CNN
+F 2 "Pin_Headers:Pin_Header_Straight_1x03" H 7250 3100 50  0001 C CNN
 F 3 "" H 7250 3100 50  0000 C CNN
 	1    7250 3100
@@
 F 0 "P6" H 2850 5500 50  0000 C CNN
 F 1 "Analog In 4" V 2950 5300 50  0000 C CNN
-F 2 "" H 2850 5300 50  0001 C CNN
+F 2 "Socket_Strips:Socket_Strip_Straight_1x03" H 2850 5300 50  0001 C CNN
 F 3 "" H 2850 5300 50  0000 C CNN
 	1    2850 5300
@@
 F 0 "P5" H 2850 4950 50  0000 C CNN
 F 1 "Analog In 3" V 2950 4750 50  0000 C CNN
-F 2 "" H 2850 4750 50  0001 C CNN
+F 2 "Socket_Strips:Socket_Strip_Straight_1x03" H 2850 4750 50  0001 C CNN
 F 3 "" H 2850 4750 50  0000 C CNN
 	1    2850 4750
@@
 F 0 "P4" H 2850 4400 50  0000 C CNN
 F 1 "Analog In 2" V 2950 4200 50  0000 C CNN
-F 2 "" H 2850 4200 50  0001 C CNN
+F 2 "Socket_Strips:Socket_Strip_Straight_1x03" H 2850 4200 50  0001 C CNN
 F 3 "" H 2850 4200 50  0000 C CNN
 	1    2850 4200
@@
 F 0 "P3" H 2850 3850 50  0000 C CNN
 F 1 "Analog In 1" V 2950 3650 50  0000 C CNN
-F 2 "" H 2850 3650 50  0001 C CNN
+F 2 "Socket_Strips:Socket_Strip_Straight_1x03" H 2850 3650 50  0001 C CNN
 F 3 "" H 2850 3650 50  0000 C CNN
 	1    2850 3650
@@
 F 0 "P2" H 2850 3300 50  0000 C CNN
 F 1 "Analog In 0" V 2950 3100 50  0000 C CNN
-F 2 "" H 2850 3100 50  0001 C CNN
+F 2 "Socket_Strips:Socket_Strip_Straight_1x03" H 2850 3100 50  0001 C CNN
 F 3 "" H 2850 3100 50  0000 C CNN
 	1    2850 3100
@@
 F 0 "P7" H 2850 6050 50  0000 C CNN
 F 1 "Analog In 5" V 2950 5850 50  0000 C CNN
-F 2 "" H 2850 5850 50  0001 C CNN
+F 2 "Socket_Strips:Socket_Strip_Straight_1x03" H 2850 5850 50  0001 C CNN
 F 3 "" H 2850 5850 50  0000 C CNN
 	1    2850 5850
@@
 Text Label 3250 5850 0    60   ~ 0
 5V
-Text Label 3950 4350 2    60   ~ 0
+Text Label 4050 2800 2    60   ~ 0
 5V
 Text Label 3100 3000 0    60   ~ 0
@@
 F 0 "LED1" H 4050 2100 50  0000 C CNN
 F 1 "Power LED" H 4050 1900 50  0000 C CNN
-F 2 "" H 4050 2000 60  0001 C CNN
+F 2 "FT:LED-1206" H 4050 2000 60  0001 C CNN
 F 3 "" H 4050 2000 60  0000 C CNN
 	1    4050 2000
@@
 F 0 "R1" V 4130 1450 50  0000 C CNN
 F 1 "150" V 4050 1450 50  0000 C CNN
-F 2 "" H 4050 1450 60  0001 C CNN
+F 2 "Resistors_SMD:R_1206_HandSoldering" H 4050 1450 60  0001 C CNN
 F 3 "" H 4050 1450 60  0000 C CNN
 	1    4050 1450
@@
 F 0 "SW1" H 6000 1260 50  0000 C CNN
 F 1 "Button 0" H 6150 1070 50  0000 C CNN
-F 2 "" H 6150 1150 60  0001 C CNN
+F 2 "Buttons_Switches_SMD:SW_SPST_PTS645" H 6150 1150 60  0001 C CNN
 F 3 "" H 6150 1150 60  0000 C CNN
 	1    6150 1150
@@
 F 0 "R2" V 7030 1150 50  0000 C CNN
 F 1 "10k" V 6950 1150 50  0000 C CNN
-F 2 "" H 6950 1150 60  0001 C CNN
+F 2 "Resistors_SMD:R_1206_HandSoldering" H 6950 1150 60  0001 C CNN
 F 3 "" H 6950 1150 60  0000 C CNN
 	1    6950 1150
@@
 F 0 "SW2" H 6000 1760 50  0000 C CNN
 F 1 "Button 1" H 6150 1570 50  0000 C CNN
-F 2 "" H 6150 1650 60  0001 C CNN
+F 2 "Buttons_Switches_SMD:SW_SPST_PTS645" H 6150 1650 60  0001 C CNN
 F 3 "" H 6150 1650 60  0000 C CNN
 	1    6150 1650
@@
 F 0 "R3" V 7030 1650 50  0000 C CNN
 F 1 "10k" V 6950 1650 50  0000 C CNN
-F 2 "" H 6950 1650 60  0001 C CNN
+F 2 "Resistors_SMD:R_1206_HandSoldering" H 6950 1650 60  0001 C CNN
 F 3 "" H 6950 1650 60  0000 C CNN
 	1    6950 1650
@@
 F 0 "SW3" H 6000 2260 50  0000 C CNN
 F 1 "Button 2" H 6150 2070 50  0000 C CNN
-F 2 "" H 6150 2150 60  0001 C CNN
+F 2 "Buttons_Switches_SMD:SW_SPST_PTS645" H 6150 2150 60  0001 C CNN
 F 3 "" H 6150 2150 60  0000 C CNN
 	1    6150 2150
@@
 F 0 "R4" V 7030 2150 50  0000 C CNN
 F 1 "10k" V 6950 2150 50  0000 C CNN
-F 2 "" H 6950 2150 60  0001 C CNN
+F 2 "Resistors_SMD:R_1206_HandSoldering" H 6950 2150 60  0001 C CNN
 F 3 "" H 6950 2150 60  0000 C CNN
 	1    6950 2150
@@
 F 0 "R5" V 8680 1150 50  0000 C CNN
 F 1 "150" V 8600 1150 50  0000 C CNN
-F 2 "" H 8600 1150 60  0001 C CNN
+F 2 "Resistors_SMD:R_1206_HandSoldering" H 8600 1150 60  0001 C CNN
 F 3 "" H 8600 1150 60  0000 C CNN
 	1    8600 1150
@@
 F 0 "LED2" H 9200 1250 50  0000 C CNN
 F 1 "Status LED" H 9200 1050 50  0000 C CNN
-F 2 "" H 9200 1150 60  0001 C CNN
+F 2 "FT:LED-1206" H 9200 1150 60  0001 C CNN
 F 3 "" H 9200 1150 60  0000 C CNN
 	1    9200 1150
@@
 NoConn ~ 6000 3650
 NoConn ~ 6000 3550
+$Comp
+L CONN_01X02 P14
+U 1 1 57FEA861
+P 4250 2850
+F 0 "P14" H 4250 3000 50  0000 C CNN
+F 1 "Power Jumper" V 4350 2850 50  0000 C CNN
+F 2 "Pin_Headers:Pin_Header_Straight_1x02" H 4250 2850 50  0001 C CNN
+F 3 "" H 4250 2850 50  0000 C CNN
+	1    4250 2850
+	1    0    0    -1
+$EndComp
+Wire Wire Line
+	3950 4350 3950 2900
+Wire Wire Line
+	3950 2900 4050 2900
 $EndSCHEMATC
